File: kicad/cnc_pendant_to_duet3D.kicad_pcb (KiCad board)
At the start: 2 copper layers, 60 x 34 mm, 9 parts, among them J1 Conn_01x04_Male, J2 DA15_Socket_MountingHoles, U1 Sparkfun_Pro_Micro

Commit message: renaming
Parts:
- J1: footprint cnc_pendant_to_duet3D:61900411021 -> cnc_pendant_to_duet3d:61900411021
- U1: footprint cnc_pendant_to_duet3D:Sparkfun_Pro_Micro -> cnc_pendant_to_duet3d:Sparkfun_Pro_Micro
Changed lines of the file:
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@@
 		(property ki_fp_filters "MountingHole*")
 		(sheetname "/")
-		(sheetfile "cnc_pendant_to_duet3D.kicad_sch")
+		(sheetfile "cnc_pendant_to_duet3d.kicad_sch")
 		(attr exclude_from_pos_files exclude_from_bom)
 		(fp_circle
@@
 		(property ki_fp_filters "R_*")
 		(sheetname "/")
-		(sheetfile "cnc_pendant_to_duet3D.kicad_sch")
+		(sheetfile "cnc_pendant_to_duet3d.kicad_sch")
 		(attr smd)
 		(fp_line
@@
 		(property ki_fp_filters "MountingHole*")
 		(sheetname "/")
-		(sheetfile "cnc_pendant_to_duet3D.kicad_sch")
+		(sheetfile "cnc_pendant_to_duet3d.kicad_sch")
 		(attr exclude_from_pos_files exclude_from_bom)
 		(fp_circle
@@
 		(property ki_fp_filters "MountingHole*")
 		(sheetname "/")
-		(sheetfile "cnc_pendant_to_duet3D.kicad_sch")
+		(sheetfile "cnc_pendant_to_duet3d.kicad_sch")
 		(attr exclude_from_pos_files exclude_from_bom)
 		(fp_circle
@@
 		(property ki_fp_filters "MountingHole*")
 		(sheetname "/")
-		(sheetfile "cnc_pendant_to_duet3D.kicad_sch")
+		(sheetfile "cnc_pendant_to_duet3d.kicad_sch")
 		(attr exclude_from_pos_files exclude_from_bom)
 		(fp_circle
@@
 		(embedded_fonts no)
 	)
-	(footprint "cnc_pendant_to_duet3D:61900411021"
+	(footprint "cnc_pendant_to_duet3d:61900411021"
 		(layer "F.Cu")
 		(at 122.65 83 -90)
@@
 		)
 		(sheetname "/")
-		(sheetfile "cnc_pendant_to_duet3D.kicad_sch")
+		(sheetfile "cnc_pendant_to_duet3d.kicad_sch")
 		(attr through_hole)
 		(fp_line
@@
 		(property ki_fp_filters "R_*")
 		(sheetname "/")
-		(sheetfile "cnc_pendant_to_duet3D.kicad_sch")
+		(sheetfile "cnc_pendant_to_duet3d.kicad_sch")
 		(attr smd)
 		(fp_line
@@
 		)
 	)
-	(footprint "cnc_pendant_to_duet3D:Sparkfun_Pro_Micro"
+	(footprint "cnc_pendant_to_duet3d:Sparkfun_Pro_Micro"
 		(layer "F.Cu")
 		(at 139 97.62 90)
@@
 		)
 		(sheetname "/")
-		(sheetfile "cnc_pendant_to_duet3D.kicad_sch")
+		(sheetfile "cnc_pendant_to_duet3d.kicad_sch")
 		(attr through_hole)
 		(fp_line
@@
 		(property ki_fp_filters "DSUB*Socket*")
 		(sheetname "/")
-		(sheetfile "cnc_pendant_to_duet3D.kicad_sch")
+		(sheetfile "cnc_pendant_to_duet3d.kicad_sch")
 		(attr through_hole)
 		(fp_line
