File: kicad/cnc_pendant_to_duet3d.kicad_pcb (KiCad board)
At the start: 2 copper layers, 60 x 34 mm, 9 parts, among them J1 Conn_01x04_Male, J2 DA15_Socket_MountingHoles, U1 Sparkfun_Pro_Micro

Commit message: Confusion over connecting to Duet and PanelDue
Change to silkscreens
Connections:
- net /io0.out renamed /DOUT
Other:
- board text added: "5v_ext"
- board text added: "dout"
- board text added: "duet"
- board text removed: "5v_ext/+5v"
- board text removed: "duet 3 io_0/ duet 2 paneldue"
- board text removed: "i0.out"
- board text removed: "i0.out/utxd0"
Changed lines of the file:
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@@
 	(net 1 "+5V")
 	(net 2 "/io0.in")
-	(net 3 "/io0.out")
+	(net 3 "/DOUT")
 	(net 4 "/Z_AXIS")
 	(net 5 "/X_AXIS")
@@
 			(layers "*.Cu" "*.Mask")
 			(remove_unused_layers no)
-			(net 3 "/io0.out")
+			(net 3 "/DOUT")
 			(pintype "passive")
 			(solder_mask_margin 0.102)
@@
 			)
 		)
-		(property "Description" "arduino pro micro"
+		(property "Description" "Sparkfun Pro Micro"
 			(at 7.62 16 0)
 			(layer "F.SilkS")
@@
 			(layers "*.Cu" "*.Mask")
 			(remove_unused_layers no)
-			(net 3 "/io0.out")
+			(net 3 "/DOUT")
 			(pinfunction "RXI")
 			(pintype "bidirectional")
@@
 		)
 	)
-	(gr_text "i0.out"
+	(gr_text "dout"
 		(at 127.3 84.8 0)
 		(layer "F.SilkS")
@@
 	)
 	(gr_text "gnd"
-		(at 126.9 82.4 0)
+		(at 126.9 82.3 0)
 		(layer "B.SilkS")
 		(effects
@@
 		)
 	)
-	(gr_text "5v_ext/+5v"
-		(at 127 87.5 0)
+	(gr_text "5v_ext"
+		(at 127 87.4 0)
 		(layer "B.SilkS")
 		(effects
@@
 		)
 	)
-	(gr_text "i0.out/utxd0"
-		(at 126.9 84.9 0)
+	(gr_text "dout"
+		(at 126.9 84.8 0)
 		(layer "B.SilkS")
 		(effects
@@
 		)
 	)
-	(gr_text "duet 3 io_0/\nduet 2 paneldue"
-		(at 122 83 270)
+	(gr_text "duet"
+		(at 128.7 77.3 0)
 		(layer "B.SilkS")
 		(effects
 			(font
 				(size 1 1)
-				(thickness 0.125)
+				(thickness 0.2)
+				(bold yes)
 			)
 			(justify bottom mirror)
